File: Kicad_Project/Custom_keyboard/Custom_keyboard.kicad_pcb (KiCad board)
At the start: 4 copper layers, 70.6 x 102.2 mm, 84 parts, among them J1 USB_C_Receptacle_USB2.0_16P, SW1 SW_Push, SW10 SW_Push, SW2 SW_Push, SW3 SW_Push, SW4 SW_Push, SW5 SW_Push, SW6 SW_Push, SW7 SW_Push, SW8 SW_Push, SW9 SW_Push, U1 RP2040, U2 USBLC6-2SC6, U3 AP2112K-3.3, U5 W25Q32JVSS, U6 SN74LV1T34DBV, Y2 Crystal_GND24

Commit message: changed board shape
Parts:
- moved D1 3.64 mm to (146.3, 75.4)
- moved R1 3.64 mm to (144.3, 72.2)
- moved R15 3.64 mm to (148.3, 75.4)
- moved R2 3.64 mm to (139.3, 72.2)
- moved R3 3.64 mm to (140.2, 79.9)
- moved R4 3.64 mm to (143.6, 79.9)
- moved U2 3.64 mm to (141.9, 75.2)
- moved J1 3.64 mm to (141.3, 65.2)
- moved C3 3.64 mm to (153.6, 71.6)
- moved C4 3.64 mm to (148.3, 72.0)
- moved F1 3.64 mm to (149.9, 68.0)
- moved U3 3.64 mm to (150.9, 72.0)
Routing:
- net VBUS: track 292.6 -> 285.5 mm
- net /D-: track 84.8 -> 81.2 mm
- net /D+: track 85.4 -> 81.8 mm
Other:
- board size 70.6 x 102.2 mm -> 70.6 x 98.5 mm
