File: Kicad_Project/Custom_keyboard/Custom_keyboard.kicad_pcb (KiCad board)
At the start: 4 copper layers, 70.6 x 98.5 mm, 84 parts, among them J1 USB_C_Receptacle_USB2.0_16P, SW1 SW_Push, SW10 SW_Push, SW2 SW_Push, SW3 SW_Push, SW4 SW_Push, SW5 SW_Push, SW6 SW_Push, SW7 SW_Push, SW8 SW_Push, SW9 SW_Push, U1 RP2040, U2 USBLC6-2SC6, U3 AP2112K-3.3, U5 W25Q32JVSS, U6 SN74LV1T34DBV, Y2 Crystal_GND24

Commit message: Use shared Kicad_Libs instead of project-specific libraries
- Project parts moved to Kicad_Libs (symbol, footprint, 3D, datasheet)
- Lib tables point to ${KIPRJMOD}/../KiCad_Libs (link via bring_libs.bat)
- Schematic/PCB references (lib ids, footprints, 3D paths, datasheets)
  updated to the Kicad_Libs libraries; no design changes
- Removed the old project-specific library folder
Parts:
- VR1, VR2: footprint PEC12R-4120F-S0012:PEC12R4120FS0012 -> eSwitch:PEC12R4120FS0012
Changed lines of the file:
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@@
 		)
 		(embedded_fonts no)
-		(model "C:/Users/lollo/Desktop/Hardware_Projects/Custom-Keyboard/3D/Kailh Polia.step"
+		(model "${KIPRJMOD}/../KiCad_Libs/eSwitch/eSwitch.3dshapes/Kailh_Polia.step"
 			(offset
 				(xyz -2.5 -5 5)
@@
 		)
 		(embedded_fonts no)
-		(model "C:/Users/lollo/Desktop/Hardware_Projects/Custom-Keyboard/3D/Kailh Polia.step"
+		(model "${KIPRJMOD}/../KiCad_Libs/eSwitch/eSwitch.3dshapes/Kailh_Polia.step"
 			(offset
 				(xyz -2.5 -5 5)
@@
 		)
 		(embedded_fonts no)
-		(model "C:/Users/lollo/Desktop/Hardware_Projects/Custom-Keyboard/3D/Kailh Polia.step"
+		(model "${KIPRJMOD}/../KiCad_Libs/eSwitch/eSwitch.3dshapes/Kailh_Polia.step"
 			(offset
 				(xyz -2.5 -5 5.5)
@@
 		)
 		(embedded_fonts no)
-		(model "C:/Users/lollo/Desktop/Hardware_Projects/Custom-Keyboard/3D/Kailh Polia.step"
+		(model "${KIPRJMOD}/../KiCad_Libs/eSwitch/eSwitch.3dshapes/Kailh_Polia.step"
 			(offset
 				(xyz -2.5 -5 5)
@@
 		)
 		(embedded_fonts no)
-		(model "C:/Users/lollo/Desktop/Hardware_Projects/Custom-Keyboard/3D/Kailh Polia.step"
+		(model "${KIPRJMOD}/../KiCad_Libs/eSwitch/eSwitch.3dshapes/Kailh_Polia.step"
 			(offset
 				(xyz -2.5 -5 5)
@@
 		)
 		(embedded_fonts no)
-		(model "C:/Users/lollo/Desktop/Hardware_Projects/Custom-Keyboard/3D/Kailh Polia.step"
+		(model "${KIPRJMOD}/../KiCad_Libs/eSwitch/eSwitch.3dshapes/Kailh_Polia.step"
 			(offset
 				(xyz -2.5 -5 5)
@@
 		)
 		(embedded_fonts no)
-		(model "C:/Users/lollo/Desktop/Hardware_Projects/Custom-Keyboard/3D/Kailh Polia.step"
+		(model "${KIPRJMOD}/../KiCad_Libs/eSwitch/eSwitch.3dshapes/Kailh_Polia.step"
 			(offset
 				(xyz -2.5 -5 5)
@@
 		)
 	)
-	(footprint "PEC12R-4120F-S0012:PEC12R4120FS0012"
+	(footprint "eSwitch:PEC12R4120FS0012"
 		(layer "F.Cu")
 		(at 118.6 86.25)
@@
 		)
 		(embedded_fonts no)
-		(model "PEC12R-4120F-S0012.stp"
+		(model "${KIPRJMOD}/../KiCad_Libs/eSwitch/eSwitch.3dshapes/PEC12R-4120F-S0012.stp"
 			(offset
 				(xyz 2.499999962 7.479999907 -0.1399999985)
@@
 		)
 	)
-	(footprint "PEC12R-4120F-S0012:PEC12R4120FS0012"
+	(footprint "eSwitch:PEC12R4120FS0012"
 		(layer "F.Cu")
 		(at 158.4 86.25)
@@
 		)
 		(embedded_fonts no)
-		(model "PEC12R-4120F-S0012.stp"
+		(model "${KIPRJMOD}/../KiCad_Libs/eSwitch/eSwitch.3dshapes/PEC12R-4120F-S0012.stp"
 			(offset
 				(xyz 2.499999962 7.479999907 -0.1399999985)
@@
 		)
 		(embedded_fonts no)
-		(model "C:/Users/lollo/Desktop/Hardware_Projects/Custom-Keyboard/3D/Kailh Polia.step"
+		(model "${KIPRJMOD}/../KiCad_Libs/eSwitch/eSwitch.3dshapes/Kailh_Polia.step"
 			(offset
 				(xyz -2.5 -5 5)
@@
 		)
 		(embedded_fonts no)
-		(model "C:/Users/lollo/Desktop/Hardware_Projects/Custom-Keyboard/3D/Kailh Polia.step"
+		(model "${KIPRJMOD}/../KiCad_Libs/eSwitch/eSwitch.3dshapes/Kailh_Polia.step"
 			(offset
 				(xyz -2.5 -5 5)
