File: Kicad_Project/Custom_keyboard/Custom_keyboard.kicad_sch (KiCad schematic)
At the start: 84 parts, among them J1 USB_C_Receptacle_USB2.0_16P, SW1 SW_Push, SW10 SW_Push, SW2 SW_Push, SW3 SW_Push, SW4 SW_Push, SW5 SW_Push, SW6 SW_Push, SW7 SW_Push, SW8 SW_Push, SW9 SW_Push, U1 RP2040, U2 USBLC6-2SC6, U3 AP2112K-3.3, U5 W25Q32JVSS, U6 SN74LV1T34DBV, Y2 Crystal_GND24

Commit message: changed board shape
Parts:
- C1, C2: LCSC (none) -> C20616249
- C10, C11, C12, C13, C16, C22, C23, C24, C25, C26, C27, C28, C29, C30, C31, C5, C6, C7, C8, C9: LCSC (none) -> C1590
- C14, C15: LCSC (none) -> C43922
- C17, C18, C19, C20: LCSC (none) -> C519406
- C21: LCSC (none) -> C91606
- C3, C4: LCSC (none) -> C5199872
- D1: LCSC (none) -> C497951
- F1: LCSC (none) -> C371166
- J1: LCSC (none) -> C3020560
- R1, R2: LCSC (none) -> C2907044
- R10, R11, R12, R13, R14, R16, R7, R8, R9: LCSC (none) -> C2906982
- R15, R5, R6: LCSC (none) -> C2907002
- R17: LCSC (none) -> C2909394
- R3, R4: LCSC (none) -> C2907136
- SW1: LCSC (none) -> C116501
- SW10, SW2, SW3, SW4, SW5, SW6, SW7, SW8, SW9: LCSC (none) -> CPG151101D01
- U1: LCSC (none) -> C2040
- U2: LCSC (none) -> C2827654
- U3: LCSC (none) -> C23380830
- U5: LCSC (none) -> C179173
- U6: LCSC (none) -> C100024
- VR1, VR2: LCSC (none) -> C143801
- Y2: LCSC (none) -> C20625731

Commit message: Use shared Kicad_Libs instead of project-specific libraries
- Project parts moved to Kicad_Libs (symbol, footprint, 3D, datasheet)
- Lib tables point to ${KIPRJMOD}/../KiCad_Libs (link via bring_libs.bat)
- Schematic/PCB references (lib ids, footprints, 3D paths, datasheets)
  updated to the Kicad_Libs libraries; no design changes
- Removed the old project-specific library folder
Parts:
- VR1, VR2: footprint PEC12R4120FS0012 -> eSwitch:PEC12R4120FS0012; symbol PEC12R-4120F-S0012:PEC12R-4120F-S0012 -> eSwitch:PEC12R-4120F-S0012
Changed lines of the file:
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@@
 	)
 	(symbol
-		(lib_id "PEC12R-4120F-S0012:PEC12R-4120F-S0012")
+		(lib_id "eSwitch:PEC12R-4120F-S0012")
 		(at 361.95 138.43 0)
 		(unit 1)
@@
 			)
 		)
-		(property "Footprint" "PEC12R4120FS0012"
+		(property "Footprint" "eSwitch:PEC12R4120FS0012"
 			(at 388.62 225.73 0)
 			(hide yes)
@@
 	)
 	(symbol
-		(lib_id "PEC12R-4120F-S0012:PEC12R-4120F-S0012")
+		(lib_id "eSwitch:PEC12R-4120F-S0012")
 		(at 367.03 201.93 0)
 		(unit 1)
@@
 			)
 		)
-		(property "Footprint" "PEC12R4120FS0012"
+		(property "Footprint" "eSwitch:PEC12R4120FS0012"
 			(at 393.7 289.23 0)
 			(hide yes)
